File: KiCad Files/MicroDev.kicad_pcb (KiCad board)
At the start: 2 copper layers, 21.5 x 11.5 mm, 13 parts, among them J1 USB_C_Receptacle_USB2.0_16P, J2 UPDI, U1 CH340E, U2 LM66100DCK

Commit message: INITIAL COMMIT
Parts:
- D1: footprint Diode_SMD:D_0402_1005Metric -> Diode_SMD:D_SOD-123
- moved D2 10.4 mm to (141.4, 78.6)
- moved R5 7.35 mm to (141.2, 80.5), turned to 0 degrees
- moved D1 1.95 mm to (136.2, 87.1)
Routing:
- net Net-(U1-TNOW): track 9.11 -> 0.00 mm, vias 2 -> 0
- net Net-(J2-Pin_2): track 17.9 -> 12.2 mm, vias 0 -> 1
- net Net-(D1-K): track 16.1 -> 11.2 mm
- net GND: track 32.7 -> 35.7 mm
- net Net-(D1-A): track 9.61 -> 10.7 mm
- net Net-(D2-A): track 1.39 -> 2.06 mm
Other:
- board text added: "1A"
- board text removed: "Rev1A"
