File: KiCad Files/MicroDev.kicad_sch (KiCad schematic)
At the start: 13 parts, among them J1 USB_C_Receptacle_USB2.0_16P, J2 UPDI, U1 CH340E, U2 LM66100DCK

Commit message: INITIAL COMMIT
Parts:
- D1: footprint Diode_SMD:D_0402_1005Metric -> Diode_SMD:D_SOD-123
Changed lines of the file:
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@@
 			)
 		)
-		(property "Footprint" "Diode_SMD:D_0402_1005Metric"
+		(property "Footprint" "Diode_SMD:D_SOD-123"
 			(at 97.79 74.93 0)
 			(hide yes)
